File: EPM3032_DEV.kicad_pcb (KiCad board)
At the start: 2 copper layers, 27.9 x 40.6 mm, 12 parts, among them J1 JTAG, J2 Conn_01x15, J3 Conn_01x15, U1 EPM3032A

Commit message: Rev2
Parts:
- added J2: Conn_01x02, Connector_PinHeader_2.54mm:PinHeader_1x02_P2.54mm_Vertical, F.Cu at (127.0, 78.7)
- R1, R2, R3, R4: value 1K -> 10K
- U1: value EPM3032A -> EPM3032A(TQFP)
- moved C3 7.96 mm to (126.4, 100.3), turned to 0 degrees
- moved C1 5.39 mm to (111.1, 91.4)
- moved C4 3.70 mm to (125.1, 88.3), turned to 0 degrees
- moved J1 2.54 mm to (121.9, 78.7)
- moved R1 2.54 mm to (119.4, 75.6)
- moved R2 2.54 mm to (116.8, 75.6)
- moved R3 2.54 mm to (121.9, 75.6)
- moved R4 2.54 mm to (111.8, 75.6)
- moved C2 0.63 mm to (113.0, 101.0), turned to 180 degrees
- renumbered J2 to J3, J3 to J4
Connections:
- J3 pad 1: /P1 -> /P2
- J3 pad 10: /P14 -> /P15
- J3 pad 11: /P16 -> /P18
- J3 pad 12: /P18 -> /P19
- J3 pad 13: /P19 -> /P20
- J3 pad 14: /P20 -> /P21
- J3 pad 15: /P21 -> /P22
- J3 pad 2: /P2 -> /P3
- J3 pad 3: /P4 -> /P5
- J3 pad 4: /P5 -> /P6
- J3 pad 5: /P6 -> /P8
- J3 pad 6: /P8 -> /P10
- J3 pad 7: /P9 -> /P12
- J3 pad 8: /P11 -> /P13
- J3 pad 9: /P12 -> /P14
- J4 pad 10: /P29 -> /P33
- J4 pad 11: /P28 -> /P31
- J4 pad 12: /P27 -> /P28
- J4 pad 13: /P26 -> /P27
- J4 pad 15: /P24 -> /P23
- J4 pad 3: /P41 -> /P42
- J4 pad 6: /P37 -> /P38
- J4 pad 7: /P34 -> /P37
- J4 pad 8: /P33 -> /P35
- J4 pad 9: /P31 -> /P34
- U1 pad 1: /P1 -> /TDI
- U1 pad 10: GND -> /P10
- U1 pad 11: /P11 -> GND
- U1 pad 13: /TMS -> /P13
- U1 pad 15: VCC -> /P15
- U1 pad 16: /P16 -> GND
- U1 pad 17: GND -> VCC
- U1 pad 22: GND -> /P22
- U1 pad 23: VCC -> /P23
- U1 pad 24: /P24 -> GND
- U1 pad 26: /P26 -> /TCK
- U1 pad 29: /P29 -> VCC
- U1 pad 3: VCC -> /P3
- U1 pad 32: /TCK -> /TDO
- U1 pad 35: VCC -> /P35
- U1 pad 38: /TDO -> /P38
- U1 pad 4: /P4 -> GND
- U1 pad 41: /P41 -> VCC
- U1 pad 42: GND -> /P42
- U1 pad 7: /TDI -> /TMS
- U1 pad 9: /P9 -> VCC
Routing:
- net /TDO: track 18.2 -> 48.1 mm, vias 1 -> 0
- net /P1: track 25.9 -> 0.00 mm, vias 1 -> 0
- net /P42: track 0.00 -> 19.1 mm
- net VCC: track 69.6 -> 87.9 mm
- net /P3: track 0.00 -> 17.3 mm
- net /P4: track 16.2 -> 0.00 mm
- net /P41: track 15.1 -> 0.00 mm
- net /P23: track 0.00 -> 13.2 mm
- net /P22: track 0.00 -> 13.2 mm
- net /P24: track 12.8 -> 0.00 mm
- net /P10: track 0.00 -> 12.1 mm, vias 0 -> 1
- net /P26: track 10.1 -> 0.00 mm
- net /P13: track 0.00 -> 9.23 mm
- net /P38: track 0.00 -> 9.08 mm
- net /P29: track 8.37 -> 0.00 mm
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Other:
- board text added: "2 3 5 6 8 10 12 13 14 15 18 19 20 21 22"
- board text added: "44 43 42 40 39 38 37 35 34 33 31 28 27 25 23"
- board text added: "GND"
- board text added: "V3.3"
- board text added: "rev2"
- board text removed: "1 2 4 5 6 8 9 11 12 14 16 18 19 20 21"
- board text removed: "44 43 41 40 39 37 34 33 31 29 28 27 26 25 24"
