File: EPM3032_DEV.kicad_sch (KiCad schematic)
At the start: 12 parts, among them J1 JTAG, J2 Conn_01x15, J3 Conn_01x15, U1 EPM3032A

Commit message: Rev2
Parts:
- removed U1: EPM3032A, Package_QFP:TQFP-44_10x10mm_P0.8mm, symbol toyoshim:EPM3032A
- added J2: Conn_01x02, Connector_PinHeader_2.54mm:PinHeader_1x02_P2.54mm_Vertical, symbol Connector_Generic:Conn_01x02
- added U1: EPM3032A(TQFP), Package_QFP:TQFP-44_10x10mm_P0.8mm, symbol toyoshim:EPM3032A(TQFP)
- R1, R2, R3, R4: value 1K -> 10K
- renumbered J2 to J3, J3 to J4
Connections:
- net P1 is gone; now on net P2: J3.1 (Pin_1)
- net P16 is gone; now on net P18: J3.11 (Pin_11)
- net P26 is gone; now on net P27: J4.13 (Pin_13)
- net P29 is gone; now on net P33: J4.10 (Pin_10)
- net P4 is gone; now on net P5: J3.3 (Pin_3)
- net P9 is gone; now on net P12: J3.7 (Pin_7)
- net GND: now also J2.2 (Pin_2), U1.11 (GND), U1.16 (GND), U1.24 (GND), U1.30 (GND), U1.36 (GND), U1.4 (GND)
- net P12: now also U1.12 (I/O); no longer J3.9 (Pin_9)
- net P14: now also J3.9 (Pin_9), U1.14 (I/O); no longer J3.10 (Pin_10)
- net P18: now also U1.18 (I/O); no longer J3.12 (Pin_12)
- net P19: now also J3.12 (Pin_12), U1.19 (I/O); no longer J3.13 (Pin_13)
- net P2: now also U1.2 (I/O); no longer J3.2 (Pin_2)
- net P20: now also J3.13 (Pin_13), U1.20 (I/O); no longer J3.14 (Pin_14)
- net P21: now also J3.14 (Pin_14), U1.21 (I/O); no longer J3.15 (Pin_15)
- net P25: now also U1.25 (I/O)
- net P27: now also U1.27 (I/O); no longer J4.12 (Pin_12)
- net P28: now also J4.12 (Pin_12), U1.28 (I/O); no longer J4.11 (Pin_11)
- net P31: now also J4.11 (Pin_11), U1.31 (I/O); no longer J4.9 (Pin_9)
- net P33: now also U1.33 (I/O); no longer J4.8 (Pin_8)
- net P34: now also J4.9 (Pin_9), U1.34 (I/O); no longer J4.7 (Pin_7)
- net P37: now also J4.7 (Pin_7), U1.37 (INPUT/GCLK1); no longer J4.6 (Pin_6)
- net P39: now also U1.39 (INPUT/GCLRn)
- net P40: now also U1.40 (INPUT/OE2/GCLK2)
- net P43: now also U1.43 (I/O)
- net P44: now also U1.44 (I/O)
- net P5: now also U1.5 (I/O); no longer J3.4 (Pin_4)
- net P6: now also J3.4 (Pin_4), U1.6 (I/O); no longer J3.5 (Pin_5)
- net P8: now also J3.5 (Pin_5), U1.8 (I/O); no longer J3.6 (Pin_6)
- net TCK: now also U1.26 (I/O/TCK)
- net TDI: now also U1.1 (I/O/TDI)
- net TDO: now also U1.32 (I/O/TDO)
- net TMS: now also U1.7 (I/O/TMS)
- net VCC: now also J2.1 (Pin_1), U1.17 (VCC), U1.29 (VCC), U1.41 (VCC), U1.9 (VCC)
- net P11 renamed P13
- net P13: now also U1.13 (I/O)
- net P24 renamed P23
- net P23: now also U1.23 (I/O)
- net P41 renamed P42
- net P42: now also U1.42 (I/O)
- new net P10: J3.6 (Pin_6), U1.10 (I/O/TMS)
- new net P15: J3.10 (Pin_10), U1.15 (I/O)
- new net P22: J3.15 (Pin_15), U1.22 (I/O)
- new net P3: J3.2 (Pin_2), U1.3 (I/O)
- new net P35: J4.8 (Pin_8), U1.35 (I/O)
- new net P38: J4.6 (Pin_6), U1.38 (INPUT/OE1)
